Commit message: fix(module): Fix paths for panda_tibia meshes

File: src/module/urdf/bonetag_tibia.in.urdf (robot description, URDF)
Before this commit: robot bonetag_tibia, 3 links, 2 joints
Links:
- link support_tibia: geometry collision mesh filename=@MODULE_INSTALL_LOCATION@/meshes/bonetag_tibia/support_tibi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 scale=0.001 0.001 0.001; visual mesh filename=@MODULE_INSTALL_LOCATION@/meshes/bonetag_tibia/support_tibi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 scale=0.001 0.001 0.001
- link tibia: geometry collision mesh filename=@MODULE_INSTALL_LOCATION@/meshes/bonetag_tibia/tibia.stl scale=0.001 0.001 0.001; visual mesh filename=@MODULE_INSTALL_LOCATION@/meshes/bonetag_tibia/tibia.stl scale=0.001 0.001 0.001
