Commit message: [modules] Generate connected modules

File: src/module/urdf/bonetag_femur.in.urdf (robot description, URDF)
Before this commit: robot bonetag_femur, 3 links, 2 joints
Links:
- link femur: geometry collision mesh filename=@MODULE_INSTALL_LOCATION@/meshes/femur.stl scale=0.001 0.001 0.001; visual mesh filename=@MODULE_INSTALL_LOCATION@/meshes/femur.stl scale=0.001 0.001 0.001

Commit message: [modules] Refactor bonetag_tibia/femur model files

File: src/module/urdf/bonetag_femur.in.urdf (robot description, URDF)
Before this commit: robot bonetag_femur, 3 links, 2 joints
Links:
- link femur: geometry collision mesh filename=@MODULE_INSTALL_LOCATION@/meshes/bonetag_femur/femur.stl scale=0.001 0.001 0.001; visual mesh filename=@MODULE_INSTALL_LOCATION@/meshes/bonetag_femur/femur.stl scale=0.001 0.001 0.001
- link support_femur: geometry collision mesh filename=@MODULE_INSTALL_LOCATION@/meshes/bonetag_femur/support_femu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 scale=0.001 0.001 0.001; visual mesh filename=@MODULE_INSTALL_LOCATION@/meshes/bonetag_femur/support_femu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 scale=0.001 0.001 0.001

Commit message: [modules] Support both panda and ur10

File: src/module/urdf/bonetag_femur.in.urdf (robot description, URDF)
Before this commit: robot bonetag_femur, 3 links, 2 joints
Links:
- removed link base_link
- added link femur_base_link
Joints:
- joint ee_to_support: parent base_link -> femur_base_link

File: src/module/urdf/bonetag_tibia.in.urdf (robot description, URDF)
Before this commit: robot bonetag_tibia, 3 links, 2 joints
Links:
- removed link base_link
- added link tibia_base_link
Joints:
- joint ee_to_support: parent base_link -> tibia_base_link

Commit message: fix(modules): Make rviz happy with file:// prefix

File: src/module/urdf/bonetag_femur.in.urdf (robot description, URDF)
Before this commit: robot bonetag_femur, 3 links, 2 joints
Links:
- link femur: geometry collision mesh filename=file://@MODULE_INSTALL_LOCATION@/meshes/bonetag_femur/femur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 scale=0.001 0.001 0.001; visual mesh filename=file://@MODULE_INSTALL_LOCATION@/meshes/bonetag_femur/femur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 scale=0.001 0.001 0.001
- link support_femur: geometry collision mesh filename=file://@MODULE_INSTALL_LOCATION@/meshes/bonetag_femur/suppo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 scale=0.001 0.001 0.001; visual mesh filename=file://@MODULE_INSTALL_LOCATION@/meshes/bonetag_femur/suppo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 scale=0.001 0.001 0.001

File: src/module/urdf/bonetag_knee_brace.in.urdf (robot description, URDF)
Before this commit: robot bonetag_knee_brace, 1 links, 0 joints
Links:
- link bonetag_knee_brace: geometry collision mesh filename=file://@MODULE_INSTALL_LOCATION@/meshes/bonetag_knee_brace/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 scale=1 1 1; visual mesh filename=file://@MODULE_INSTALL_LOCATION@/meshes/bonetag_knee_brace/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 scale=1 1 1

File: src/module/urdf/bonetag_tibia.in.urdf (robot description, URDF)
Before this commit: robot bonetag_tibia, 3 links, 2 joints
Links:
- link support_tibia: geometry collision mesh filename=file://@MODULE_INSTALL_LOCATION@/meshes/bonetag_tibia/suppo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 scale=0.001 0.001 0.001; visual mesh filename=file://@MODULE_INSTALL_LOCATION@/meshes/bonetag_tibia/suppo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 scale=0.001 0.001 0.001
- link tibia: geometry collision mesh filename=file://@MODULE_INSTALL_LOCATION@/meshes/bonetag_tibia/tibia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 scale=0.001 0.001 0.001; visual mesh filename=file://@MODULE_INSTALL_LOCATION@/meshes/bonetag_tibia/tibia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 scale=0.001 0.001 0.001

File: src/module/urdf/bonetag_tibia_calibration_tool.in.urdf (robot description, URDF)
Before this commit: robot bonetag_tibia_calibration_tool, 1 links, 0 joints
Links:
- link bonetag_tibia_calibration_tool: geometry collision mesh filename=file://@MODULE_INSTALL_LOCATION@/meshes/bonetag_tibia/calib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 scale=0.001 0.001 0.001; visual mesh filename=file://@MODULE_INSTALL_LOCATION@/meshes/bonetag_tibia/calib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 scale=0.001 0.001 0.001

File: src/module/urdf/taa_talar.in.urdf (robot description, URDF)
Before this commit: robot taa_talar, 1 links, 0 joints
Links:
- link taa_talar: geometry collision mesh filename=file://@MODULE_INSTALL_LOCATION@/meshes/taa_talar/taa_talar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 scale=0.001 0.001 0.001; visual mesh filename=file://@MODULE_INSTALL_LOCATION@/meshes/taa_talar/taa_talar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 scale=0.001 0.001 0.001

File: src/module/urdf/taa_tibia.in.urdf (robot description, URDF)
Before this commit: robot taa_tibia, 1 links, 0 joints
Links:
- link taa_tibia: geometry collision mesh filename=file://@MODULE_INSTALL_LOCATION@/meshes/taa_tibia/taa_tibia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 scale=0.001 0.001 0.001; visual mesh filename=file://@MODULE_INSTALL_LOCATION@/meshes/taa_tibia/taa_tibia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 scale=0.001 0.001 0.001
